File: PCB/Waveform_Gen_ADSR.kicad_pcb (KiCad board)
At the start: 2 copper layers, 50.8 x 22.9 mm, 28 parts, among them J6 WAVE_OUT, M1 Feather_M4_Express, U1 AD9833, U2 LMV116, U3 AD5245, X1 ASV-25.000MHZ-E-T

Commit message: working on layout
Parts:
- moved G*** 26.3 mm to (90.0, 108.2)
- moved G*** 21.1 mm to (83.2, 108.1)
- moved U3 15.7 mm to (128.1, 103.6), turned to 270 degrees
- moved R6 15.4 mm to (129.2, 99.8)
- moved R7 15.0 mm to (126.4, 99.8)
- moved C5 9.66 mm to (103.1, 111.6), turned to 180 degrees
- moved X1 8.31 mm to (108.8, 110.4)
- moved C1 8.14 mm to (113.8, 106.5), turned to 270 degrees
- moved D1 5.82 mm to (105.3, 99.1)
- moved C3 4.63 mm to (121.1, 103.0), turned to 270 degrees
- moved C11 4.45 mm to (116.2, 106.5)
- moved L1 3.80 mm to (119.1, 111.1)
- moved L2 3.80 mm to (119.1, 113.6)
- moved C7 3.67 mm to (116.1, 112.3)
- moved C6 3.33 mm to (113.9, 112.3)
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Routing:
- net Net-(D1-Pad2): track 15.7 -> 0.00 mm
- net Net-(C4-Pad1): track 22.4 -> 10.1 mm
- net Net-(U2-Pad3): track 0.00 -> 12.0 mm
- net /25MHZ_CLK: track 9.11 -> 19.0 mm
- net +3V3: track 45.3 -> 37.2 mm
- net +3.3VA: track 32.0 -> 38.6 mm
- net GND: track 4.08 -> 0.00 mm
- net /~WAVE_CS: track 14.1 -> 16.2 mm
- net Net-(C1-Pad1): track 8.61 -> 10.7 mm
- net GNDA: track 3.96 -> 5.31 mm, vias 7 -> 6
- net /SCLK: track 10.4 -> 11.2 mm
- net Net-(C10-Pad1): track 18.0 -> 18.7 mm
- removed copper zone on B.Cu, net GND
- removed copper zone on F.Cu, net GND

Commit message: update layout
Parts:
- R1: moved to F.Cu
- moved R1 16.1 mm to (114.7, 102.5)
- moved C2 11.1 mm to (134.3, 103.7), turned to 180 degrees
- moved R6 10.9 mm to (118.3, 100.1), turned to 180 degrees
- moved R7 8.57 mm to (118.2, 102.5), turned to 180 degrees
- moved R4 7.50 mm to (139.9, 106.2), turned to 180 degrees
- moved C10 4.32 mm to (134.3, 106.2)
- moved C1 4.31 mm to (118.1, 105.8), turned to 180 degrees
- moved U1 4.19 mm to (128.8, 108.3)
- moved C9 4.16 mm to (125.4, 112.1)
- moved C3 4.01 mm to (123.3, 106.3), turned to 90 degrees
- moved C8 3.72 mm to (123.3, 112.1)
- moved C11 2.54 mm to (118.1, 108.2), turned to 180 degrees
- moved C4 2.47 mm to (134.3, 101.6), turned to 0 degrees
- moved C5 1.98 mm to (104.6, 110.3), turned to 270 degrees
- moved L2 1.46 mm to (120.5, 113.2)
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Routing:
- net Net-(J6-Pad1): track 25.4 -> 0.00 mm
- net +3.3VA: track 38.6 -> 15.8 mm, vias 2 -> 0
- net Net-(C10-Pad1): track 18.7 -> 0.00 mm
- net /~WAVE_CS: track 16.2 -> 0.00 mm, vias 1 -> 0
- net +3V3: track 37.2 -> 52.6 mm
- net Net-(U2-Pad3): track 12.0 -> 0.00 mm
- net /SCLK: track 11.2 -> 0.00 mm, vias 1 -> 0
- net Net-(C4-Pad1): track 10.1 -> 0.00 mm
- net /MOSI: track 9.61 -> 0.00 mm, vias 1 -> 0
- net /POT_SDA: track 0.00 -> 9.43 mm, vias 0 -> 1
- net /POT_SCL: track 0.00 -> 8.09 mm, vias 0 -> 1
- net GNDA: track 5.31 -> 0.00 mm, vias 6 -> 5
- net Net-(C3-Pad2): track 3.25 -> 5.52 mm
- net /25MHZ_CLK: track 19.0 -> 17.2 mm
- net /WAVE_OUT: track 18.1 -> 19.4 mm
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- removed copper zone on B.Cu, net GNDA
- removed copper zone on F.Cu, net GNDA

Commit message: update layout
Parts:
- moved C10 5.14 mm to (133.2, 111.2)
- moved R5 3.33 mm to (130.1, 112.8)
- moved D1 3.00 mm to (105.5, 102.1)
- moved G*** 1.32 mm to (82.2, 108.9)
- moved C3 0.94 mm to (123.3, 105.4)
- moved C11 0.63 mm to (118.1, 107.6)
- moved C1 0.30 mm to (118.1, 105.5)
Routing:
- net Net-(J6-Pad1): track 0.00 -> 41.0 mm
- net /~WAVE_CS: track 0.00 -> 37.4 mm, vias 0 -> 1
- net /POT_SDA: track 9.43 -> 33.6 mm
- net GND: track 0.00 -> 23.2 mm, vias 7 -> 9
- net /POT_SCL: track 8.09 -> 28.6 mm
- net +3.3VA: track 15.8 -> 33.0 mm
- net Net-(U2-Pad3): track 0.00 -> 15.6 mm
- net Net-(C10-Pad1): track 0.00 -> 14.0 mm
- net +3V3: track 52.6 -> 66.5 mm
- net Net-(C4-Pad1): track 0.00 -> 10.1 mm
- net GNDA: track 0.00 -> 5.85 mm, vias 5 -> 6
- net /25MHZ_CLK: track 17.2 -> 20.9 mm
- net /WAVE_OUT: track 19.4 -> 22.4 mm
- net Net-(C1-Pad1): track 9.99 -> 11.2 mm
- added copper zone on B.Cu, net GNDA
- added copper zone on F.Cu, net GNDA

Commit message: update layout
Parts:
- R5: moved to B.Cu
- U1: footprint Housings_SSOP:MSOP-10_3x3mm_Pitch0.5mm -> Housings_SSOP:MSOP-10-1EP_3x3mm_Pitch0.5mm
- moved D1 14.0 mm to (96.6, 91.3)
- moved R5 3.72 mm to (133.4, 114.4), turned to 0 degrees
- moved C1 3.62 mm to (115.2, 107.7), turned to 270 degrees
- moved R1 2.96 mm to (114.5, 99.5)
- moved R6 2.43 mm to (116.5, 101.8)
- moved R7 2.43 mm to (116.5, 104.1)
- moved G*** 1.04 mm to (82.5, 109.9)
- moved C10 0.99 mm to (133.3, 112.2)
- moved U3 0.88 mm to (128.5, 102.2), turned to 0 degrees
- moved C11 0.85 mm to (117.2, 107.7), turned to 270 degrees
- moved C3 0.64 mm to (123.9, 105.6), turned to 0 degrees
Routing:
- net Net-(J6-Pad1): track 41.0 -> 25.8 mm
- net /SCLK: track 0.00 -> 12.3 mm
- net +3.3VA: track 33.0 -> 43.2 mm, vias 0 -> 3
- net /MOSI: track 0.00 -> 8.41 mm, vias 0 -> 2
- net /POT_SDA: track 33.6 -> 40.2 mm
- net GNDA: track 5.85 -> 0.00 mm
- net /POT_SCL: track 28.6 -> 34.4 mm
- net Net-(C10-Pad1): track 14.0 -> 19.8 mm
- net /WAVE_OUT: track 22.4 -> 17.6 mm, vias 1 -> 0
- net /~WAVE_CS: track 37.4 -> 41.8 mm
- net GND: track 23.2 -> 18.8 mm
- net Net-(C3-Pad2): track 5.62 -> 3.25 mm
- net +3V3: track 66.5 -> 64.6 mm
- net Net-(C4-Pad1): track 10.1 -> 11.2 mm
- net Net-(C1-Pad1): track 11.2 -> 12.3 mm
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- added copper zone on B.Cu, net GND
- added copper zone on F.Cu, net GND

Commit message: update PCB layout
Parts:
- U1: value AD9833 -> AD9833/37
- moved G*** 17.2 mm to (99.4, 106.8)
- moved D1 14.4 mm to (105.6, 102.5)
- moved G*** 9.58 mm to (99.5, 106.7)
- moved R5 1.69 mm to (134.0, 112.8)
- moved C10 0.78 mm to (133.8, 111.6), turned to 270 degrees
Routing:
- net Net-(D1-Pad2): track 0.00 -> 13.2 mm, vias 0 -> 1
- net GNDA: track 0.00 -> 5.55 mm, vias 6 -> 7
- net /POT_SCL: track 34.4 -> 38.7 mm
- net GND: track 18.8 -> 22.9 mm, vias 9 -> 12
- net /POT_SDA: track 40.2 -> 43.9 mm
- net /SCLK: track 12.3 -> 15.8 mm, vias 0 -> 1
- net /WAVE_OUT: track 17.6 -> 21.1 mm
- net Net-(J6-Pad1): track 25.8 -> 23.8 mm
- net Net-(C10-Pad1): track 19.8 -> 21.5 mm
- net /MOSI: track 8.41 -> 9.27 mm, vias 2 -> 0
- net /~WAVE_CS: track 41.8 -> 41.1 mm
- net Net-(C1-Pad1): track 12.3 -> 13.0 mm
Other:
- board text added: "WAVE_OUT -> A0"
- board text removed: "WAVE_OUT"

Commit message: update layout; stack AD983x footprints
Parts:
- added U4: AD9837, Housings_CSP:AD9837BCPZ-RL7, F.Cu at (128.8, 108.3)
- U1: value AD9833/37 -> AD9833; footprint Housings_SSOP:MSOP-10-1EP_3x3mm_Pitch0.5mm -> Housings_SSOP:MSOP-10_3x3mm_Pitch0.5mm
Connections:
- net Net-(C1-Pad1) renamed /CAP
- net Net-(C3-Pad2) renamed /COMP
- net Net-(C4-Pad1) renamed /VOUT
Routing:
- net /SCLK: track 15.8 -> 16.8 mm
- net /MOSI: track 9.27 -> 10.2 mm
- net GNDA: track 5.55 -> 6.39 mm
- net /VOUT: track 11.2 -> 12.0 mm
- net /~WAVE_CS: track 41.1 -> 41.9 mm
- net GND: track 22.9 -> 23.6 mm
- net /25MHZ_CLK: track 20.9 -> 21.6 mm
- net /COMP: track 3.25 -> 3.92 mm
- net /CAP: track 13.0 -> 13.6 mm
Other:
- board text added: "WAVE_OUT -> A2"
- board text removed: "WAVE_OUT -> A0"

Commit message: update pcb layout; add stacked footprints; add sine logo
Parts:
- added G***: SINE, Adafruit:WAVE_GEN_SINE_LOGO, F.Cu at (99.4, 106.8)
- moved G*** 39.2 mm to (138.6, 105.9)

Commit message: update PCB layout; include support for AD9837
Parts:
- moved G*** 33.5 mm to (105.4, 110.0)
Other:
- board text added: "AD9833/37 Precision Waveform Generator + 8-bit amplitude control (via I2C) + FeatherWing, 3.3v powered + DC to 1MHz, 0.1Hz accuracy + Sine/Square/Triangle waveform + 3.3v buffered output + SPI interface for waveform gen (D6 = ~CS~)"
- board text removed: "AD9833 Precision Waveform Generator + 8-bit amplitude control (via I2C) + FeatherWing, 3.3v powered + DC to 1MHz, 0.1Hz accuracy + Sine/Square/Triangle waveform + 3.3v buffered output + SPI interface for waveform gen (D6 = ~CS~)"
Changed lines of the file:
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@@
   (general
     (thickness 1.6)
-    (drawings 59)
+    (drawings 58)
     (tracks 286)
     (zones 0)
@@
   )
   (module Adafruit:WAVE_GEN_LOGO (layer B.Cu)
-    (at 138.63 105.87 180)
+    (at 105.41 109.982 180)
     (fp_text reference G*** (at 0 4.5 180) (layer B.SilkS) hide
       (effects (font (size 0.5 0.5) (thickness 0.1)) (justify mirror))
@@
       (xy -1.060246 -1.792306) (xy -0.950167 -1.797256) (xy -0.86098 -1.779418)) (layer F.Mask) (width 0.01))
   )
-  (gr_poly (pts (xy 101.64 104.63) (xy 97.34 104.63) (xy 97.34 108.96) (xy 101.65 108.96)) (layer B.Mask) (width 0.15))
+  (gr_text "Amplitude\nControl" (at 108.077 114.046) (layer B.SilkS)
+    (effects (font (size 0.6 0.6) (thickness 0.1)) (justify left mirror))
+  )
   (gr_line (start 119.888 114.3) (end 123.19 114.3) (layer B.SilkS) (width 0.1))
   (gr_line (start 145.415 99.695) (end 145.288 99.695) (layer F.SilkS) (width 0.1))
@@
   (gr_line (start 141.605 114.3) (end 141.605 113.665) (layer B.SilkS) (width 0.1))
   (gr_poly (pts (xy 124.2314 110.3122) (xy 124.2314 110.0622) (xy 124.4814 110.0622) (xy 124.4814 110.3122)) (layer F.SilkS) (width 0.15))
-  (gr_text "Amplitude\nControl" (at 141.88 101.91) (layer B.SilkS)
-    (effects (font (size 0.6 0.6) (thickness 0.1)) (justify left mirror))
-  )
   (gr_line (start 120.7 112.6) (end 120.5 112.6) (layer F.SilkS) (width 0.1))
   (gr_line (start 120.4 113.8) (end 120.7 112.6) (layer F.SilkS) (width 0.1))
@@
     (effects (font (size 0.6 0.6) (thickness 0.1)) (justify mirror))
   )
-  (gr_text "AD9833 Precision Waveform Generator\n  + 8-bit amplitude control (via I2C)\n  + FeatherWing, 3.3v powered\n  + DC to 1MHz, 0.1Hz accuracy\n  + Sine/Square/Triangle waveform\n  + 3.3v buffered output\n  + SPI interface for waveform\n         gen (D6 = ~CS~)" (at 135.27 105.87) (layer B.SilkS)
+  (gr_text "AD9833/37 Precision Waveform Generator\n  + 8-bit amplitude control (via I2C)\n  + FeatherWing, 3.3v powered\n  + DC to 1MHz, 0.1Hz accuracy\n  + Sine/Square/Triangle waveform\n  + 3.3v buffered output\n  + SPI interface for waveform gen (D6 = ~CS~)" (at 140.208 104.648) (layer B.SilkS)
     (effects (font (size 0.5 0.5) (thickness 0.1)) (justify left mirror))
   )
-  (gr_text 2019-09-09v00 (at 140.37 113.22) (layer B.SilkS)
+  (gr_text 2019-09-09v00 (at 125.476 108.712) (layer B.SilkS)
     (effects (font (size 0.5 0.5) (thickness 0.1)) (justify mirror))
   )
@@
   (gr_arc (start 144.145 116.205) (end 144.145 118.11) (angle -90) (layer Edge.Cuts) (width 0.1))
   (gr_arc (start 144.145 97.155) (end 146.05 97.155) (angle -90) (layer Edge.Cuts) (width 0.1))
-  (gr_text "ANALOG SECTION" (at 138.43 99.695) (layer B.SilkS)
+  (gr_text "ANALOG SECTION" (at 126.492 113.665) (layer B.SilkS)
     (effects (font (size 0.5 0.5) (thickness 0.1)) (justify left mirror))
   )
@@
       )
     )
-  )
-  (zone (net 0) (net_name "") (layer F.Cu) (hatch edge 0.508)
-    (connect_pads (clearance 0.254))
-    (min_thickness 0.254)
-    (keepout (tracks not_allowed) (vias not_allowed) (copperpour not_allowed))
-    (fill (arc_segments 16) (thermal_gap 0.508) (thermal_bridge_width 0.508))
-    (polygon
-      (pts
-        (xy 97.39 106.45) (xy 97.54 106.07) (xy 97.79 105.57) (xy 97.97 105.29) (xy 98.14 105.12)
-        (xy 98.25 105.04) (xy 98.44 105) (xy 98.61 105.03) (xy 98.75 105.15) (xy 98.9 105.35)
-        (xy 99.12 105.76) (xy 99.51 106.74) (xy 99.97 107.88) (xy 100.13 108.2) (xy 100.3 108.41)
-        (xy 100.42 108.48) (xy 100.51 108.48) (xy 100.61 108.45) (xy 100.73 108.36) (xy 100.87 108.19)
-        (xy 101 107.96) (xy 101.19 107.6) (xy 101.36 107.16) (xy 101.48 106.87) (xy 101.53 106.83)
-        (xy 101.64 106.83) (xy 101.65 106.88) (xy 101.5 107.22) (xy 101.27 107.78) (xy 101.07 108.16)
-        (xy 100.81 108.48) (xy 100.63 108.64) (xy 100.5 108.66) (xy 100.37 108.65) (xy 100.27 108.6)
-        (xy 100.19 108.55) (xy 100.09 108.42) (xy 99.98 108.24) (xy 99.84 107.97) (xy 99.63 107.51)
-        (xy 99.51 107.2) (xy 99.36 106.79) (xy 99.19 106.38) (xy 99.02 105.95) (xy 98.92 105.73)
-        (xy 98.82 105.53) (xy 98.73 105.37) (xy 98.64 105.27) (xy 98.56 105.2) (xy 98.52 105.17)
-        (xy 98.43 105.16) (xy 98.36 105.17) (xy 98.29 105.2) (xy 98.21 105.25) (xy 98.14 105.33)
-        (xy 97.99 105.53) (xy 97.86 105.78) (xy 97.72 106.08) (xy 97.57 106.44) (xy 97.44 106.76)
-        (xy 97.43 106.83) (xy 97.24 106.83) (xy 97.3 106.66)
-      )
-    )
-  )
-  (zone (net 0) (net_name "") (layer B.Cu) (hatch edge 0.508)
-    (connect_pads (clearance 0.254))
-    (min_thickness 0.254)
-    (keepout (tracks allowed) (vias not_allowed) (copperpour not_allowed))
-    (fill (arc_segments 16) (thermal_gap 0.508) (thermal_bridge_width 0.508))
-    (polygon
-      (pts
-        (xy 96.97 106.99) (xy 97.25 106.07) (xy 97.64 105.29) (xy 98.13 104.78) (xy 98.6 104.72)
-        (xy 98.805 104.845) (xy 99.1 105.17) (xy 99.32 105.56) (xy 99.87 106.91) (xy 100.17 107.74)
-        (xy 100.48 108.23) (xy 100.7 107.94) (xy 101.011869 107.286102) (xy 101.36 106.56) (xy 101.97 106.64)
-        (xy 101.84 107.14) (xy 101.38 108.22) (xy 100.85 108.85) (xy 100.51 108.97) (xy 100.01 108.78)
-        (xy 99.62 108.22) (xy 98.71 105.82) (xy 98.41 105.43) (xy 98.06 105.92) (xy 97.55 107.1)
-      )
-    )
