File: PCB/Waveform_Gen_ADSR.sch (KiCad schematic (older format))
At the start: 26 parts, among them J6 WAVE_OUT, M1 Feather_M4_Express, U1 AD9833, U2 LMV116, U3 AD5245, X1 ASV-25.000MHZ-E-T

Commit message: working on layout
Parts:
- U1: footprint Housings_SSOP:MSOP-10_3x3mm_Pitch0.5mm -> Housings_SSOP:MSOP-10-1EP_3x3mm_Pitch0.5mm
Changed lines of the file:
@@
 F 0 "U1" H 5075 2075 50  0000 L CNN
 F 1 "AD9833" H 4900 1975 50  0000 L CNN
-F 2 "Housings_SSOP:MSOP-10_3x3mm_Pitch0.5mm" H 5225 2075 25  0001 C CNN
+F 2 "Housings_SSOP:MSOP-10-1EP_3x3mm_Pitch0.5mm" H 5225 2075 25  0001 C CNN
 F 3 "" H 4475 2725 50  0001 C CNN
 	1    4575 2725

Commit message: update PCB layout
Other:
- note added: "TANT"
Changed lines of the file:
@@
 Text Notes 1200 2375 0    50   ~ 0
 Consider a note for AD9837's lower clock speed
+Text Notes 4100 1550 0    50   ~ 0
+TANT
+Text Notes 8600 5925 0    50   ~ 0
+TANT
 $EndSCHEMATC

Commit message: update layout; stack AD983x footprints
Parts:
- added U4: AD9837BCPZ-RL7, Housings_CSP:AD9837BCPZ-RL7, symbol AD9837BCPZ-RL7:AD9837BCPZ-RL7
- U1: footprint Housings_SSOP:MSOP-10-1EP_3x3mm_Pitch0.5mm -> Housings_SSOP:MSOP-10_3x3mm_Pitch0.5mm
Connections:
- net labels added: CAP, COMP, VOUT
- wire segments 124 -> 137
Other:
- note added: "ALTERNATE FOOTPRINT"
- note removed: "Change footprint to include AD9837's grounding pad"

Commit message: update PCB layout; include support for AD9837
Other:
- note added: "AD9837: ASV-16.000MHZ-E-T"
- note added: "Alternate Wave Gen\nFootprint"
- note added: "Envelope\nPotentiometer"
- note removed: "ALTERNATE FOOTPRINT"
- note removed: "Consider a note for AD9837's lower clock speed"

Commit message: change scope to support only AD9833
Parts:
- removed U4: AD9837BCPZ-RL7, Housings_CSP:AD9837BCPZ-RL7, symbol AD9837BCPZ-RL7:AD9837BCPZ-RL7
Connections:
- wire segments 137 -> 124
Other:
- note removed: "AD9837: ASV-16.000MHZ-E-T"
- note removed: "Alternate Wave Gen\nFootprint"
Changed lines of the file:
@@
 Sheet 1 1
 Title "ADSR_Waveform_Generator"
-Date "2019-09-10"
+Date "2019-09-13"
 Rev "v00"
 Comp "Cedar Grove Studios"
@@
 Text Notes 7825 1475 0    50   ~ 0
 GAIN_BW = 45MHz\n9.75MHz BW at gain of 4.6\n
-Text Notes 3025 5475 0    50   ~ 0
-Alternate Wave Gen\nFootprint
-Text Notes 1825 3100 0    50   ~ 0
-AD9837: ASV-16.000MHZ-E-T
 Text Notes 3575 950  0    50   ~ 0
 TANT
 Text Notes 3725 7225 0    50   ~ 0
 TANT
-$Comp
-L AD9837BCPZ-RL7:AD9837BCPZ-RL7 U4
-U 1 1 5D78AAF8
-P 2750 4300
-F 0 "U4" H 3400 3875 60  0000 L CNN
-F 1 "AD9837BCPZ-RL7" H 3375 3775 60  0000 L CNN
-F 2 "Housings_CSP:AD9837BCPZ-RL7" H 4150 4540 60  0001 C CNN
-F 3 "" H 2750 4300 60  0000 C CNN
-	1    2750 4300
-	1    0    0    -1
-$EndComp
 Wire Wire Line
 	2700 2025 3250 2025
@@
 Text Label 3900 1375 1    50   ~ 0
 CAP
-$Comp
-L power:GND #PWR0123
-U 1 1 5D7BF4F0
-P 2550 5300
-F 0 "#PWR0123" H 2550 5050 50  0001 C CNN
-F 1 "GND" H 2555 5127 50  0000 C CNN
-F 2 "" H 2550 5300 50  0001 C CNN
-F 3 "" H 2550 5300 50  0001 C CNN
-	1    2550 5300
-	1    0    0    -1
-$EndComp
-$Comp
-L power:GNDA #PWR0124
-U 1 1 5D7BF4F6
-P 2850 5300
-F 0 "#PWR0124" H 2850 5050 50  0001 C CNN
-F 1 "GNDA" H 2855 5127 50  0000 C CNN
-F 2 "" H 2850 5300 50  0001 C CNN
-F 3 "" H 2850 5300 50  0001 C CNN
-	1    2850 5300
-	1    0    0    -1
-$EndComp
-Wire Wire Line
-	2850 5300 2850 5275
-Wire Wire Line
-	2550 5300 2550 5200
-$Comp
-L power:+3.3VA #PWR0125
-U 1 1 5D7C3EFC
-P 2850 3575
-F 0 "#PWR0125" H 2850 3425 50  0001 C CNN
-F 1 "+3.3VA" H 2865 3748 50  0000 C CNN
-F 2 "" H 2850 3575 50  0001 C CNN
-F 3 "" H 2850 3575 50  0001 C CNN
-	1    2850 3575
-	1    0    0    -1
-$EndComp
-Text Label 1500 4100 0    50   ~ 0
-SCLK
-Text Label 1500 4200 0    50   ~ 0
-MOSI
-Text Label 1500 4300 0    50   ~ 0
-~WAVE_CS
-Wire Wire Line
-	1500 4300 1900 4300
-Wire Wire Line
-	1500 4200 1900 4200
-Wire Wire Line
-	1500 4100 1900 4100
-Text Label 1500 4900 0    50   ~ 0
-25MHZ_CLK
-Text Label 3800 4400 2    50   ~ 0
-VOUT
-Text Label 3800 4100 2    50   ~ 0
-COMP
-Text Label 2550 3600 1    50   ~ 0
-CAP
-Wire Wire Line
-	3500 4400 3800 4400
-Wire Wire Line
-	3500 4100 3800 4100
-Wire Wire Line
-	2850 3650 2850 3575
-Wire Wire Line
-	2550 3450 2550 3650
-Wire Wire Line
-	1500 4900 1900 4900
-Wire Wire Line
-	3150 5200 3150 5275
-Wire Wire Line
-	3150 5275 2850 5275
-Connection ~ 2850 5275
-Wire Wire Line
-	2850 5275 2850 5200
 Text Notes 4675 4425 0    50   ~ 0
 Envelope\nPotentiometer

Commit message: update photos and board design files
Other:
- note added: "GAIN_BW = 45MHz\n9.75MHz BW at gain of 4.6\nPractical range from 0.5Hz to 100kHz\n"
- note removed: "GAIN_BW = 45MHz\n9.75MHz BW at gain of 4.6\n"
Changed lines of the file:
@@
 $EndComp
 Text Notes 7825 1475 0    50   ~ 0
-GAIN_BW = 45MHz\n9.75MHz BW at gain of 4.6\n
+GAIN_BW = 45MHz\n9.75MHz BW at gain of 4.6\nPractical range from 0.5Hz to 100kHz\n
 Text Notes 3575 950  0    50   ~ 0
 TANT
